Commit message: Release v1.3.0

File: fanuc_hardware_interface/config/6dof_robot_physical_ros2_control_macro.xacro (robot description, xacro)
@@ -42,4 +42,5 @@
         <param name="out_cmd_interp_buff_target">$(arg out_cmd_interp_buff_target)</param>
         <param name="force_sensor_type">$(arg force_sensor_type)</param>
+        <param name="motion_control">$(arg motion_control)</param>
       </hardware>
     </ros2_control>

File: fanuc_hardware_interface/config/crx_physical_ros2_control_macro.xacro (robot description, xacro)
@@ -42,4 +42,5 @@
         <param name="out_cmd_interp_buff_target">$(arg out_cmd_interp_buff_target)</param>
         <param name="force_sensor_type">$(arg force_sensor_type)</param>
+	<param name="motion_control">$(arg motion_control)</param>
       </hardware>
     </ros2_control>

File: fanuc_hardware_interface/robot/6dof_robot.urdf.xacro (robot description, xacro)
@@ -11,6 +11,12 @@
   <xacro:arg name="force_sensor_type" default="0"/>
   <xacro:arg name="use_mock" default="false"/>
-  <xacro:property name="tmpaaa" default="fanuc_$(arg robot_series)_description"/>
-  <xacro:include filename="$(find ${tmpaaa})/urdf/$(arg robot_model)_urdf_macro.xacro"/>
+  <xacro:arg name="motion_control" default="1"/>
+  <xacro:arg name="origin_xyz" default="0 0 0"/>
+  <xacro:arg name="origin_rpy" default="0 0 0"/>
+  <xacro:arg name="parent_link" default="world"/>
+  <xacro:arg name="child_link" default="end_effector"/>
+  <xacro:arg name="prefix" default="" />
+  <xacro:property name="robot_description_name" default="fanuc_$(arg robot_series)_description"/>
+  <xacro:include filename="$(find ${robot_description_name})/urdf/$(arg robot_model)_urdf_macro.xacro"/>
   <xacro:if value="$(arg use_mock)">
     <xacro:include filename="$(find fanuc_hardware_interface)/config/6dof_robot_mock_ros2_control_macro.xacro"/>
@@ -19,9 +25,9 @@
     <xacro:include filename="$(find fanuc_hardware_interface)/config/6dof_robot_physical_ros2_control_macro.xacro"/>
   </xacro:unless>
-  <link name="world"/>
-  <link name="end_effector"/>
-  <xacro:call macro="$(arg robot_model)" parent="world" child="end_effector">
-    <origin xyz="0 0 0" rpy="0 0 0"/>
+  <link name="$(arg parent_link)"/>
+  <link name="$(arg child_link)"/>
+  <xacro:call macro="$(arg robot_model)" parent="$(arg parent_link)" child="$(arg child_link)" prefix="$(arg prefix)">
+    <origin xyz="$(arg origin_xyz)" rpy="$(arg origin_rpy)"/>
   </xacro:call>
-  <xacro:robot_control name="$(arg robot_model)"/>
+  <xacro:robot_control name="$(arg robot_model)" prefix="$(arg prefix)"/>
 </robot>

File: fanuc_hardware_interface/robot/crx10ia.urdf.xacro (robot description, xacro)
@@ -9,4 +9,10 @@
   <xacro:arg name="force_sensor_type" default="1"/>
   <xacro:arg name="use_mock" default="false"/>
+  <xacro:arg name="motion_control" default="1"/>
+  <xacro:arg name="origin_xyz" default="0 0 0"/>
+  <xacro:arg name="origin_rpy" default="0 0 0"/>
+  <xacro:arg name="parent_link" default="world"/>
+  <xacro:arg name="child_link" default="end_effector"/>
+  <xacro:arg name="prefix" default="" />
   <xacro:include filename="$(find fanuc_crx_description)/urdf/crx10ia_urdf_macro.xacro"/>
   <xacro:if value="$(arg use_mock)">
@@ -16,9 +22,9 @@
     <xacro:include filename="$(find fanuc_hardware_interface)/config/crx_physical_ros2_control_macro.xacro"/>
   </xacro:unless>
-  <link name="world"/>
-  <link name="end_effector"/>
-  <xacro:crx10ia parent="world" child="end_effector">
-    <origin xyz="0 0 0" rpy="0 0 0"/>
+  <link name="$(arg parent_link)"/>
+  <link name="$(arg child_link)"/>
+  <xacro:crx10ia parent="$(arg parent_link)" child="$(arg child_link)" prefix="$(arg prefix)">
+    <origin xyz="$(arg origin_xyz)" rpy="$(arg origin_rpy)"/>
   </xacro:crx10ia>
-  <xacro:crx_control name="crx10ia"/>
+  <xacro:crx_control name="crx10ia"  prefix="$(arg prefix)"/>
 </robot>

File: fanuc_hardware_interface/robot/crx10ia_l.urdf.xacro (robot description, xacro)
@@ -9,4 +9,10 @@
   <xacro:arg name="force_sensor_type" default="1"/>
   <xacro:arg name="use_mock" default="false"/>
+  <xacro:arg name="motion_control" default="1"/>
+  <xacro:arg name="origin_xyz" default="0 0 0"/>
+  <xacro:arg name="origin_rpy" default="0 0 0"/>
+  <xacro:arg name="parent_link" default="world"/>
+  <xacro:arg name="child_link" default="end_effector"/>
+  <xacro:arg name="prefix" default="" />
   <xacro:include filename="$(find fanuc_crx_description)/urdf/crx10ia_l_urdf_macro.xacro"/>
   <xacro:if value="$(arg use_mock)">
@@ -16,9 +22,9 @@
     <xacro:include filename="$(find fanuc_hardware_interface)/config/crx_physical_ros2_control_macro.xacro"/>
   </xacro:unless>
-  <link name="world"/>
-  <link name="end_effector"/>
-  <xacro:crx10ia_l parent="world" child="end_effector">
-    <origin xyz="0 0 0" rpy="0 0 0"/>
+  <link name="$(arg parent_link)"/>
+  <link name="$(arg child_link)"/>
+  <xacro:crx10ia_l parent="$(arg parent_link)" child="$(arg child_link)" prefix="$(arg prefix)">
+    <origin xyz="$(arg origin_xyz)" rpy="$(arg origin_rpy)"/>
   </xacro:crx10ia_l>
-  <xacro:crx_control name="crx10ia_l"/>
+  <xacro:crx_control name="crx10ia_l" prefix="$(arg prefix)"/>
 </robot>

File: fanuc_hardware_interface/robot/crx20ia_l.urdf.xacro (robot description, xacro)
@@ -9,4 +9,10 @@
   <xacro:arg name="force_sensor_type" default="1"/>
   <xacro:arg name="use_mock" default="false"/>
+  <xacro:arg name="motion_control" default="1"/>
+  <xacro:arg name="origin_xyz" default="0 0 0"/>
+  <xacro:arg name="origin_rpy" default="0 0 0"/>
+  <xacro:arg name="parent_link" default="world"/>
+  <xacro:arg name="child_link" default="end_effector"/>
+  <xacro:arg name="prefix" default="" />
   <xacro:include filename="$(find fanuc_crx_description)/urdf/crx20ia_l_urdf_macro.xacro"/>
   <xacro:if value="$(arg use_mock)">
@@ -16,9 +22,9 @@
     <xacro:include filename="$(find fanuc_hardware_interface)/config/crx_physical_ros2_control_macro.xacro"/>
   </xacro:unless>
-  <link name="world"/>
-  <link name="end_effector"/>
-  <xacro:crx20ia_l parent="world" child="end_effector">
-    <origin xyz="0 0 0" rpy="0 0 0"/>
+  <link name="$(arg parent_link)"/>
+  <link name="$(arg child_link)"/>
+  <xacro:crx20ia_l parent="$(arg parent_link)" child="$(arg child_link)" prefix="$(arg prefix)">
+    <origin xyz="$(arg origin_xyz)" rpy="$(arg origin_rpy)"/>
   </xacro:crx20ia_l>
-  <xacro:crx_control name="crx20ia_l"/>
+  <xacro:crx_control name="crx20ia_l"  prefix="$(arg prefix)"/>
 </robot>

File: fanuc_hardware_interface/robot/crx30ia.urdf.xacro (robot description, xacro)
@@ -9,4 +9,10 @@
   <xacro:arg name="force_sensor_type" default="1"/>
   <xacro:arg name="use_mock" default="false"/>
+  <xacro:arg name="motion_control" default="1"/>
+  <xacro:arg name="origin_xyz" default="0 0 0"/>
+  <xacro:arg name="origin_rpy" default="0 0 0"/>
+  <xacro:arg name="parent_link" default="world"/>
+  <xacro:arg name="child_link" default="end_effector"/>
+  <xacro:arg name="prefix" default="" />
   <xacro:include filename="$(find fanuc_crx_description)/urdf/crx30ia_urdf_macro.xacro"/>
   <xacro:if value="$(arg use_mock)">
@@ -16,9 +22,9 @@
     <xacro:include filename="$(find fanuc_hardware_interface)/config/crx_physical_ros2_control_macro.xacro"/>
   </xacro:unless>
-  <link name="world"/>
-  <link name="end_effector"/>
-  <xacro:crx30ia parent="world" child="end_effector">
-    <origin xyz="0 0 0" rpy="0 0 0"/>
+  <link name="$(arg parent_link)"/>
+  <link name="$(arg child_link)"/>
+  <xacro:crx30ia parent="$(arg parent_link)" child="$(arg child_link)" prefix="$(arg prefix)">
+    <origin xyz="$(arg origin_xyz)" rpy="$(arg origin_rpy)"/>
   </xacro:crx30ia>
-  <xacro:crx_control name="crx30ia"/>
+  <xacro:crx_control name="crx30ia"  prefix="$(arg prefix)"/>
 </robot>

File: fanuc_hardware_interface/robot/crx3ia.urdf.xacro (robot description, xacro)
@@ -9,4 +9,10 @@
   <xacro:arg name="force_sensor_type" default="1"/>
   <xacro:arg name="use_mock" default="false"/>
+  <xacro:arg name="motion_control" default="1"/>
+  <xacro:arg name="origin_xyz" default="0 0 0"/>
+  <xacro:arg name="origin_rpy" default="0 0 0"/>
+  <xacro:arg name="parent_link" default="world"/>
+  <xacro:arg name="child_link" default="end_effector"/>
+  <xacro:arg name="prefix" default="" />
   <xacro:include filename="$(find fanuc_crx_description)/urdf/crx3ia_urdf_macro.xacro"/>
   <xacro:if value="$(arg use_mock)">
@@ -16,9 +22,9 @@
     <xacro:include filename="$(find fanuc_hardware_interface)/config/crx_physical_ros2_control_macro.xacro"/>
   </xacro:unless>
-  <link name="world"/>
-  <link name="end_effector"/>
-  <xacro:crx3ia parent="world" child="end_effector">
-    <origin xyz="0 0 0" rpy="0 0 0"/>
+  <link name="$(arg parent_link)"/>
+  <link name="$(arg child_link)"/>
+  <xacro:crx3ia parent="$(arg parent_link)" child="$(arg child_link)" prefix="$(arg prefix)">
+    <origin xyz="$(arg origin_xyz)" rpy="$(arg origin_rpy)"/>
   </xacro:crx3ia>
-  <xacro:crx_control name="crx3ia"/>
+  <xacro:crx_control name="crx3ia" prefix="$(arg prefix)"/>
 </robot>

File: fanuc_hardware_interface/robot/crx5ia.urdf.xacro (robot description, xacro)
@@ -9,4 +9,10 @@
   <xacro:arg name="force_sensor_type" default="1"/>
   <xacro:arg name="use_mock" default="false"/>
+  <xacro:arg name="motion_control" default="1"/>
+  <xacro:arg name="origin_xyz" default="0 0 0"/>
+  <xacro:arg name="origin_rpy" default="0 0 0"/>
+  <xacro:arg name="parent_link" default="world"/>
+  <xacro:arg name="child_link" default="end_effector"/>
+  <xacro:arg name="prefix" default="" />
   <xacro:include filename="$(find fanuc_crx_description)/urdf/crx5ia_urdf_macro.xacro"/>
   <xacro:if value="$(arg use_mock)">
@@ -16,9 +22,9 @@
     <xacro:include filename="$(find fanuc_hardware_interface)/config/crx_physical_ros2_control_macro.xacro"/>
   </xacro:unless>
-  <link name="world"/>
-  <link name="end_effector"/>
-  <xacro:crx5ia parent="world" child="end_effector">
-    <origin xyz="0 0 0" rpy="0 0 0"/>
+  <link name="$(arg parent_link)"/>
+  <link name="$(arg child_link)"/>
+  <xacro:crx5ia parent="$(arg parent_link)" child="$(arg child_link)" prefix="$(arg prefix)">
+    <origin xyz="$(arg origin_xyz)" rpy="$(arg origin_rpy)"/>
   </xacro:crx5ia>
-  <xacro:crx_control name="crx5ia"/>
+  <xacro:crx_control name="crx5ia" prefix="$(arg prefix)"/>
 </robot>
